File: hardware/remote.kicad_pcb (KiCad board)
At the start: 2 copper layers, 40 x 25 mm, 27 parts, among them J1 Debug, P1 CON-SENSOR2, P2 BOOT, U1 XMC1302-32, U2 RFM69HW, U3 DRILL, U4 DRILL, U5 DRILL, U6 DRILL

Commit message: Add new 3d model with more detailed components
Parts:
- U2: footprint RFM69HW -> kicad-libraries:RFM69HW
